File: REV3n/mainboard_REV3n/PowerMeter new Teensy4_1_Rev3n.kicad_pcb (KiCad board)
At the start: 2 copper layers, 129.6 x 89.8 mm, 52 parts, among them J1 Conn_02x05_Odd_Even, J10 RJ45_Amphenol_RJMG1BD3B8K1ANR, J11 Conn_01x04_Socket, J12 Conn_02x20_Odd_Even, J5 Conn_01x10_Socket, J7 Conn_01x02_Socket, K1 FRT5, Q1 MMBT3904, Q2 MMBT3904, U10 ISL60002DIH326Z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

Commit message: Add files via upload
Connections:
- J1 pad 2: +5V -> GNDD
- J1 pad 3: GNDD -> CS0
- J1 pad 4: GNDD -> CS1
Routing:
- net +5V: track 353.2 -> 355.0 mm
- net GNDD: vias 283 -> 295
- net GND: vias 5 -> 0
- net (no net): vias 0 -> 5
