File: REV3n/mainboard_REV3n/PowerMeter new Teensy4_1_Rev3n.kicad_sch (KiCad schematic)
At the start: 48 parts, among them J1 Conn_02x05_Odd_Even, J10 RJ45_Amphenol_RJMG1BD3B8K1ANR, J11 Conn_01x04_Socket, J12 Conn_02x20_Odd_Even, J5 Conn_01x10_Socket, J7 Conn_01x02_Socket, K1 FRT5, Q1 MMBT3904, Q2 MMBT3904, U10 ISL60002DIH326Z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

Commit message: Add files via upload
Connections:
- net +5V: no longer J1.2 (Pin_2)
- net GNDD: now also J1.2 (Pin_2); no longer J1.3 (Pin_3), J1.4 (Pin_4)
- new net CS0: J1.3 (Pin_3)
- new net CS1: J1.4 (Pin_4)
Other:
- note added: "add CS0/CS1 on J1"
