File: REV3n/mainboard_REV3n/PowerMeter_REV36.kicad_sch (KiCad schematic)
At the start: 73 parts, among them J1 Extender Board, J11 PTT IN/OUT, J2 Conn_02x08_Odd_Even, J3 Conn_02x05_Odd_Even, J4 Conn_Coaxial, J7 POWER CON, K1 FRT5, Q1 MMBT3904, Q2 MMBT3904, SW1 CK_KMS2xxGP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

Commit message: Add files via upload
Parts:
- C34, C39: value 100uF -> 10uF
Changed lines of the file:
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@@
 			)
 		)
-		(property "Value" "100uF"
+		(property "Value" "10uF"
 			(at 152.4 58.8009 0)
 			(effects
@@
 			)
 		)
-		(property "Value" "100uF"
+		(property "Value" "10uF"
 			(at 186.69 201.0409 0)
 			(effects
