File: REV3n/extender_REV3n/PowerMeter new Teensy4_1_REV3n_extender.kicad_pcb (KiCad board)
At the start: 2 copper layers, 50 x 60 mm, 54 parts, among them J13 UFL, J14 SMA, J15 UFL, J16 UFL, J17 SMA, J18 Conn_01x02_Socket, J19 Conn_01x02_Socket, J20 Conn_02x05_Odd_Even, J6 UFL, U11 PE4259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

Commit message: Add files via upload
Connections:
- J20 pad 1: +5V -> GNDD
- J20 pad 3: GNDD -> CS1
- J20 pad 4: GNDD -> CS0
Routing:
- net GNDD: track 10.6 -> 3.61 mm
- net +5V: track 83.8 -> 85.7 mm
Other:
- board text added: "REV3.2"
- board text removed: "REV1.0"
