File: REV3n/extender_REV3n/PowerMeter new Teensy4_1_REV3n_extender.kicad_sch (KiCad schematic)
At the start: 54 parts, among them J13 UFL, J14 SMA, J15 UFL, J16 UFL, J17 SMA, J18 Conn_01x02_Socket, J19 Conn_01x02_Socket, J20 Conn_02x05_Odd_Even, J6 UFL, U11 PE4259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

Commit message: Add files via upload
Connections:
- net +5V: no longer J20.1 (Pin_1)
- net GNDD: now also J20.1 (Pin_1); no longer J20.3 (Pin_3), J20.4 (Pin_4)
- new net CS0: J20.4 (Pin_4)
- new net CS1: J20.3 (Pin_3)
Other:
- note added: "add CS0/CS1 on J20"
