File: RF-Coupler/RF-Coupler HF-6m/PowerMeter_REV3n_RF_coupler1to70.kicad_pcb (KiCad board)
At the start: 2 copper layers, 55 x 80 mm, 25 parts

Commit message: Add files via upload
Parts:
- removed C1, C2: 15p, Capacitor_SMD:C_1206_3216Metric_Pad1.33x1.80mm_HandSolder
- removed L1, L2, L3, L4: 82nH, Inductor_SMD:L_1210_3225Metric_Pad1.42x2.65mm_HandSolder
- removed R13: 200R, Resistor_SMD:R_2512_6332Metric_Pad1.40x3.35mm_HandSolder
- removed R14: 200R, Resistor_SMD:R_1206_3216Metric_Pad1.30x1.75mm_HandSolder
- R1, R2, R3, R4, R6, R7, R8, R9: value 200R -> 130R
- R10, R12, R5: value 200R -> 390R
- R11: value 200R -> 390R; footprint Resistor_SMD:R_1206_3216Metric_Pad1.30x1.75mm_HandSolder -> Resistor_SMD:R_2512_6332Metric_Pad1.40x3.35mm_HandSolder
- moved R12 40.3 mm to (139.2, 99.0), turned to -90 degrees
- moved R8 11.8 mm to (109.5, 92.0), turned to 90 degrees
- moved R11 7.41 mm to (112.5, 96.9), turned to 0 degrees
- moved R9 1.52 mm to (109.5, 101.9)
- moved R3 1.32 mm to (147.2, 76.4)
- moved R4 0.92 mm to (147.2, 80.3)
Connections:
- R1 pad 2: Net-(L1-Pad1) -> GND
- R11 pad 2: Net-(L4-Pad1) -> Net-(R1-Pad1)
- R12 pad 1: Net-(R1-Pad1) -> Net-(R12-Pad1)
- R12 pad 2: Net-(L1-Pad1) -> Net-(REF1-Pin_1)
- R2 pad 2: Net-(L1-Pad1) -> GND
- R3 pad 1: Net-(R13-Pad1) -> Net-(R12-Pad1)
- R3 pad 2: Net-(L2-Pad1) -> GND
- R4 pad 1: Net-(R13-Pad1) -> Net-(R12-Pad1)
- R4 pad 2: Net-(L2-Pad1) -> GND
- R5 pad 1: Net-(R13-Pad1) -> Net-(R12-Pad1)
- R6 pad 2: Net-(L3-Pad1) -> GND
- R7 pad 2: Net-(L3-Pad1) -> GND
- R8 pad 2: Net-(L4-Pad1) -> GND
- R9 pad 2: Net-(L4-Pad1) -> GND
Routing:
- net Net-(R13-Pad1): track 24.5 -> 0.00 mm
- net Net-(R12-Pad1): track 0.00 -> 23.1 mm
- net Net-(L4-Pad1): track 10.6 -> 0.00 mm
- net Net-(FWD1-Pin_1): track 19.9 -> 11.8 mm
- net Net-(L2-Pad1): track 7.98 -> 0.00 mm
- net Net-(L3-Pad1): track 7.98 -> 0.00 mm
- net Net-(L1-Pad1): track 7.90 -> 0.00 mm
- net GND: track 0.00 -> 0.20 mm, vias 535 -> 587
Other:
- board text added: "RF-Coupler 1Mhz - 60Mhz REV 1.2"
- board text removed: "RF-Coupler 1Mhz - 60Mhz REV 1.0"
