File: RF-Coupler/RF-Coupler HF-6m/PowerMeter_REV3n_RF_coupler1to70.kicad_sch (KiCad schematic)
At the start: 26 parts, among them T1 L_Coupled, T2 L_Coupled

Commit message: Add files via upload
Parts:
- removed C1, C2: 15p, Capacitor_SMD:C_1206_3216Metric_Pad1.33x1.80mm_HandSolder, symbol Device:C
- removed L1, L2, L3, L4: 82nH, Inductor_SMD:L_1210_3225Metric_Pad1.42x2.65mm_HandSolder, symbol Device:L
- removed R13: 200R, Resistor_SMD:R_2512_6332Metric_Pad1.40x3.35mm_HandSolder, symbol Device:R
- removed R14: 200R, Resistor_SMD:R_1206_3216Metric_Pad1.30x1.75mm_HandSolder, symbol Device:R
- R1, R2, R3, R4, R6, R7, R8, R9: value 200R -> 130R
- R10, R12, R5: value 200R -> 390R
- R11: value 200R -> 390R; footprint Resistor_SMD:R_1206_3216Metric_Pad1.30x1.75mm_HandSolder -> Resistor_SMD:R_2512_6332Metric_Pad1.40x3.35mm_HandSolder
Connections:
- net GND: now also R1.2, R2.2, R3.2, R4.2, R6.2, R7.2, R8.2, R9.2
- net at R1.1, R10.2, R2.1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: now also R11.2; no longer R12.1
- net at R3.1, R4.1, R5.1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: now also R12.1
- net at R5.2, R6.1, R7.1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: now also R12.2
Other:
- note added: "-18db PAD"
